Commit message: baxter related changes

File: baxter/baxter_moveit_config/config/baxter.srdf.xacro (robot description, xacro)
@@ -1,10 +1,10 @@
 <?xml version="1.0" ?>
 <robot name="baxter" xmlns:xacro="http://www.ros.org/wiki/xacro">
-  <xacro:arg name="left_tip_name" default="left_gripper"/>
+  <!-- <xacro:arg name="left_tip_name" default="left_gripper"/> -->
   <xacro:arg name="right_tip_name" default="right_gripper"/>
   <xacro:include filename="$(find baxter_moveit_config)/config/baxter_base.srdf.xacro" />
-  <xacro:baxter_base left_tip_name="$(arg left_tip_name)" right_tip_name="$(arg right_tip_name)"/>
+  <xacro:baxter_base right_tip_name="$(arg right_tip_name)"/>
   <!--Left End Effector Collisions-->
-  <xacro:include filename="$(find baxter_moveit_config)/config/default_gripper.srdf.xacro" />
+  <!-- <xacro:include filename="$(find baxter_moveit_config)/config/default_gripper.srdf.xacro" />
   <xacro:default_gripper side="left"/>
   <xacro:arg name="left_electric_gripper" default="false"/>
@@ -12,5 +12,5 @@
     <xacro:include filename="$(find baxter_moveit_config)/config/rethink_electric_gripper.srdf.xacro" />
     <xacro:rethink_electric_gripper side="left"/>
-  </xacro:if>
+  </xacro:if> -->
   <!--Right End Effector Collisions-->
   <xacro:include filename="$(find baxter_moveit_config)/config/default_gripper.srdf.xacro" />

File: baxter/baxter_moveit_config/config/baxter_base.srdf.xacro (robot description, xacro)
@@ -5,5 +5,5 @@
 -->
 <robot xmlns:xacro="http://www.ros.org/wiki/xacro" name="baxter">
-  <xacro:macro name="baxter_base" params="left_tip_name right_tip_name">
+  <xacro:macro name="baxter_base" params="right_tip_name">
     <!--GROUPS: Representation of a set of joints and links. This can be useful for specifying DOF to plan for, defining arms, end effectors, etc-->
     <!--LINKS: When a link is specified, the parent joint of that link (if it exists) is automatically included-->
@@ -11,9 +11,9 @@
     <!--CHAINS: When a chain is specified, all the links along the chain (including endpoints) are included in the group. Additionally, all the joints that are parents to included links are also included. This means that joints along the chain and the parent joint of the base link are included in the group-->
     <!--SUBGROUPS: Groups can also be formed by referencing to already defined group names-->
-    <xacro:arg name="left_tip_name" default="left_gripper"/>
+    <!-- <xacro:arg name="left_tip_name" default="left_gripper"/> -->
     <xacro:arg name="right_tip_name" default="right_gripper"/>
-    <group name="left_arm">
+    <!-- <group name="left_arm">
         <chain base_link="torso" tip_link="$(arg left_tip_name)" />
-    </group>
+    </group> -->
     <group name="right_arm">
         <chain base_link="torso" tip_link="$(arg right_tip_name)" />
@@ -21,17 +21,17 @@
     <group name="both_arms">
         <group name="right_arm" />
-        <group name="left_arm" />
+        <!-- <group name="left_arm" /> -->
     </group>
-    <group name="left_hand">
+    <!-- <group name="left_hand">
         <chain base_link="left_hand" tip_link="$(arg left_tip_name)" />
-    </group>
+    </group> -->
     <group name="right_hand">
         <chain base_link="right_hand" tip_link="$(arg right_tip_name)" />
     </group>
     <!--END EFFECTOR: Purpose: Represent information about an end effector.-->
-    <end_effector name="left_hand_eef" parent_link="$(arg left_tip_name)" group="left_hand" parent_group="left_arm" />
+    <!-- <end_effector name="left_hand_eef" parent_link="$(arg left_tip_name)" group="left_hand" parent_group="left_arm" /> -->
     <end_effector name="right_hand_eef" parent_link="$(arg right_tip_name)" group="right_hand" parent_group="right_arm" />
     <!--GROUP STATES: Purpose: Define a named state for a particular group, in terms of joint values. This is useful to define states like 'folded arms'-->
-    <group_state name="left_neutral" group="left_arm">
+    <!-- <group_state name="left_neutral" group="left_arm">
         <joint name="left_e0" value="0" />
         <joint name="left_e1" value="0.75" />
@@ -41,5 +41,5 @@
         <joint name="left_w1" value="1.26" />
         <joint name="left_w2" value="0" />
-    </group_state>
+    </group_state> -->
     <group_state name="right_neutral" group="right_arm">
         <joint name="right_e0" value="0" />
@@ -59,7 +59,7 @@
     <disable_collisions link1="collision_head_link_1" link2="collision_head_link_2" reason="Adjacent" />
     <disable_collisions link1="collision_head_link_1" link2="head" reason="Never" />
-    <disable_collisions link1="collision_head_link_1" link2="left_lower_shoulder" reason="Never" />
+    <!-- <disable_collisions link1="collision_head_link_1" link2="left_lower_shoulder" reason="Never" />
     <disable_collisions link1="collision_head_link_1" link2="left_upper_elbow" reason="Never" />
-    <disable_collisions link1="collision_head_link_1" link2="left_upper_shoulder" reason="Never" />
+    <disable_collisions link1="collision_head_link_1" link2="left_upper_shoulder" reason="Never" /> -->
     <disable_collisions link1="collision_head_link_1" link2="pedestal" reason="Never" />
     <disable_collisions link1="collision_head_link_1" link2="right_upper_elbow_visual" reason="Never" />
@@ -71,5 +71,5 @@
     <disable_collisions link1="collision_head_link_1" link2="display" reason="Adjacent" />
     <disable_collisions link1="collision_head_link_2" link2="head" reason="Never" />
-    <disable_collisions link1="collision_head_link_2" link2="left_upper_shoulder" reason="Never" />
+    <!-- <disable_collisions link1="collision_head_link_2" link2="left_upper_shoulder" reason="Never" /> -->
     <disable_collisions link1="collision_head_link_2" link2="pedestal" reason="Never" />
     <disable_collisions link1="collision_head_link_2" link2="right_lower_shoulder" reason="Never" />
@@ -80,10 +80,10 @@
     <disable_collisions link1="collision_head_link_2" link2="torso" reason="Adjacent" />
     <disable_collisions link1="collision_head_link_2" link2="display" reason="Adjacent" />
-    <disable_collisions link1="head" link2="left_hand_camera" reason="Never" />
+    <!-- <disable_collisions link1="head" link2="left_hand_camera" reason="Never" />
     <disable_collisions link1="head" link2="left_hand_range" reason="Never" />
     <disable_collisions link1="head" link2="left_lower_shoulder" reason="Never" />
     <disable_collisions link1="head" link2="left_upper_elbow" reason="Never" />
     <disable_collisions link1="head" link2="left_upper_elbow_visual" reason="Never" />
-    <disable_collisions link1="head" link2="left_upper_shoulder" reason="Never" />
+    <disable_collisions link1="head" link2="left_upper_shoulder" reason="Never" /> -->
     <disable_collisions link1="head" link2="pedestal" reason="Never" />
     <disable_collisions link1="head" link2="right_hand_camera" reason="Never" />
@@ -96,5 +96,5 @@
     <disable_collisions link1="head" link2="sonar_ring" reason="Never" />
     <disable_collisions link1="head" link2="torso" reason="Adjacent" />
-    <disable_collisions link1="left_hand" link2="left_hand_camera" reason="Adjacent" />
+    <!-- <disable_collisions link1="left_hand" link2="left_hand_camera" reason="Adjacent" />
     <disable_collisions link1="left_hand" link2="left_hand_range" reason="Adjacent" />
     <disable_collisions link1="left_hand" link2="left_lower_elbow" reason="Never" />
@@ -191,5 +191,5 @@
     <disable_collisions link1="left_upper_shoulder" link2="screen" reason="Never" />
     <disable_collisions link1="left_upper_shoulder" link2="sonar_ring" reason="Never" />
-    <disable_collisions link1="left_upper_shoulder" link2="torso" reason="Adjacent" />
+    <disable_collisions link1="left_upper_shoulder" link2="torso" reason="Adjacent" /> -->
     <disable_collisions link1="pedestal" link2="right_hand_accelerometer" reason="Never" />
     <disable_collisions link1="pedestal" link2="right_hand_camera" reason="Default" />
@@ -201,5 +201,5 @@
     <disable_collisions link1="pedestal" link2="right_upper_forearm_visual" reason="Default" />
     <disable_collisions link1="pedestal" link2="right_upper_shoulder" reason="Never" />
-    <disable_collisions link1="pedestal" link2="left_hand_accelerometer" reason="Never" />
+    <!-- <disable_collisions link1="pedestal" link2="left_hand_accelerometer" reason="Never" />
     <disable_collisions link1="pedestal" link2="left_hand_camera" reason="Default" />
     <disable_collisions link1="pedestal" link2="left_hand_range" reason="Default" />
@@ -209,5 +209,5 @@
     <disable_collisions link1="pedestal" link2="left_upper_forearm" reason="Never" />
     <disable_collisions link1="pedestal" link2="left_upper_forearm_visual" reason="Default" />
-    <disable_collisions link1="pedestal" link2="left_upper_shoulder" reason="Never" />
+    <disable_collisions link1="pedestal" link2="left_upper_shoulder" reason="Never" /> -->
     <disable_collisions link1="pedestal" link2="screen" reason="Never" />
     <disable_collisions link1="pedestal" link2="sonar_ring" reason="Never" />
